Commit message: działa, jest nowe gui, kolejny krok to kamera i ewentualnie docker

File: urdf/ramie.urdf (robot description, URDF)
Before this commit: robot moje_ramie, 9 links, 8 joints
Links:
- removed link arm
- removed link base
- removed link end_effector
- removed link forearm
- removed link gripper_base
- removed link left_finger
- removed link right_finger
- added link arm_link; collision cylinder length=0.6 radius=0.05; visual cylinder length=0.6 radius=0.05
- added link elbow_link; collision cylinder length=0.1 radius=0.05; visual cylinder length=0.1 radius=0.05
- added link forearm_link; collision cylinder length=0.5 radius=0.05; visual cylinder length=0.5 radius=0.05
- added link gripper_base_link; collision box size=0.2 0.06 0.02; visual box size=0.2 0.06 0.02
- added link gripper_left_finger_link; collision box size=0.02 0.06 0.08; visual box size=0.02 0.06 0.08
- added link gripper_right_finger_link; collision box size=0.02 0.06 0.08; visual box size=0.02 0.06 0.08
- added link hand_link; collision box size=0.1 0.1 0.02; visual box size=0.1 0.1 0.02
- added link shoulder_link; collision cylinder length=0.5 radius=0.1; visual cylinder length=0.5 radius=0.1
- added link tool_link
- added link wrist_link; collision box size=0.1 0.1 0.05; visual box size=0.1 0.1 0.05
- link base_link: geometry collision box size=0.4 0.4 0.1; visual box size=0.4 0.4 0.1
- link hand: mass 0.5 -> None; geometry 
Joints:
- removed joint arm_to_forearm
- removed joint base_joint
- removed joint base_to_arm
- removed joint forearm_to_hand
- removed joint gripper_left_joint
- removed joint gripper_right_joint
- removed joint hand_to_end_effector
- removed joint hand_to_gripper_base
- added joint arm_to_gripper: type fixed, parent tool_link, child gripper_base_link, origin xyz=0 0 0 rpy=0 0 0
- added joint gripper_left_finger_joint: type prismatic, parent gripper_base_link, child gripper_left_finger_link, origin xyz=-0.07 0 0.02 rpy=0 0 0, axis 1 0 0, limit lower=0.0 upper=0.06 effort=1000.0 velocity=1.0
- added joint gripper_right_finger_joint: type prismatic, parent gripper_base_link, child gripper_right_finger_link, origin xyz=0.07 0 0.02 rpy=0 0 0, axis 1 0 0, limit lower=-0.06 upper=0.0 effort=1000.0 velocity=1.0, mimic joint=gripper_left_finger_joint multiplier=-1
- added joint gripper_to_hand_center: type fixed, parent gripper_base_link, child hand, origin xyz=0 0 0.06 rpy=0 0 0
- added joint hand_tool_joint: type fixed, parent hand_link, child tool_link, origin xyz=0 0 0.02 rpy=0 0 0
- added joint joint1: type revolute, parent base_link, child shoulder_link, origin xyz=0 0 0.1 rpy=0 0 0, axis 0 0 1, limit lower=-3.14 upper=3.14 effort=1000.0 velocity=1.0
- added joint joint2: type revolute, parent shoulder_link, child arm_link, origin xyz=0 0 0.5 rpy=0 0 0, axis 0 1 0, limit lower=-2.5 upper=2.5 effort=1000.0 velocity=1.0
- added joint joint3: type revolute, parent arm_link, child elbow_link, origin xyz=0 0 0.6 rpy=0 0 0, axis 0 1 0, limit lower=-2.5 upper=2.5 effort=1000.0 velocity=1.0
- added joint joint4: type revolute, parent elbow_link, child forearm_link, origin xyz=0 0 0.1 rpy=0 0 0, axis 0 0 1, limit lower=-3.14 upper=3.14 effort=1000.0 velocity=1.0
- added joint joint5: type revolute, parent forearm_link, child wrist_link, origin xyz=0 0 0.5 rpy=0 0 0, axis 0 1 0, limit lower=-1.57 upper=1.57 effort=1000.0 velocity=1.0
- added joint joint6: type continuous, parent wrist_link, child hand_link, origin xyz=0 0 0.05 rpy=0 0 0, axis 0 0 1

Commit message: przregulowania i osobne stosy plus ich liczenie trzeba oggarnąć

File: urdf/ramie.urdf (robot description, URDF)
Before this commit: robot ramie_z_chwytakiem, 12 links, 11 joints
Links:
- link arm_link: mass None -> 2.0
- link base_link: mass None -> 10.0
- link elbow_link: mass None -> 0.5
- link forearm_link: mass None -> 1.5
- link gripper_base_link: mass None -> 0.3
- link gripper_left_finger_link: mass None -> 0.1
- link gripper_right_finger_link: mass None -> 0.1
- link hand_link: mass None -> 0.2
- link shoulder_link: mass None -> 5.0
- link wrist_link: mass None -> 0.5
